File: design/CNC Boosterpack.sch (KiCad schematic (older format))
At the start: 64 parts, among them J1 JP1, J10 EEPROMaddr, J11 UART/GPIO, J2 JP2, J3 JP3, J4 I2CDrv, J5 I2C, J6 RESET, J7 VDrvGND, J8 VDrvSel, J9 Spindle/Coolant, P1 CONN_02x10, P12 YA, P13 YB, P14 ZA, P15 ZB, P17 VMOT, P2 GPIO, P3 Control, P6 XB, P7 CONN_02x10, P8 Limits, P9 XA, Q1 2N7002, Q2 2N7002, Q3 2N7002, Q4 2N7002, U1 TLP290-4, U2 TLP290-4, U3 TLP290-4, U4 24LC16, U5 TCA9406

Commit message: Updated to latest revision
A small batch of the Trinamic-version PCB has been made, driver
development in good progress. Marlin-style M-commands will be supported
including status reports. Grbl protocol extensions allows real-trime
plotting of data (stallguard value) for simpler tuning.
Parts:
- added P10: ZMotor, IoEngineering:PinHeader_1x04_P2.54mm_Vertical_Motor, symbol Connector_Generic:Conn_01x04
- added P11: Limits, Connector_PinHeader_2.54mm:PinHeader_2x02_P2.54mm_Vertical, symbol Connector_Generic:Conn_02x02_Odd_Even
- added P4: XMotor, IoEngineering:PinHeader_1x04_P2.54mm_Vertical_Motor, symbol Connector_Generic:Conn_01x04
- added P5: YMotor, IoEngineering:PinHeader_1x04_P2.54mm_Vertical_Motor, symbol Connector_Generic:Conn_01x04
- J12: renamed from R14; value 0R -> 0; footprint Resistor_SMD:R_0805_2012Metric -> Jumper:SolderJumper-2_P1.3mm_Open_RoundedPad1.0x1.5mm; symbol Device:R -> Connector_Generic:Conn_01x02
- J13: renamed from R10; value 0R -> 0; footprint Resistor_SMD:R_0805_2012Metric -> Jumper:SolderJumper-2_P1.3mm_Open_RoundedPad1.0x1.5mm; symbol Device:R -> Connector_Generic:Conn_01x02
- J14: renamed from R11; value 0R -> 0; footprint Resistor_SMD:R_0805_2012Metric -> Jumper:SolderJumper-2_P1.3mm_Open_RoundedPad1.0x1.5mm; symbol Device:R -> Connector_Generic:Conn_01x02
- J15: renamed from R13; value 0R -> 0; footprint Resistor_SMD:R_0805_2012Metric -> Jumper:SolderJumper-2_P1.3mm_Open_RoundedPad1.0x1.5mm; symbol Device:R -> Connector_Generic:Conn_01x02
- J16: renamed from R12; value 0R -> 0; footprint Resistor_SMD:R_0805_2012Metric -> Jumper:SolderJumper-2_P1.3mm_Open_RoundedPad1.0x1.5mm; symbol Device:R -> Connector_Generic:Conn_01x02
- J9: footprint Connector_PinHeader_2.54mm:PinHeader_1x07_P2.54mm_Vertical -> Connector_PinHeader_2.54mm:PinHeader_2x06_P2.54mm_Vertical; symbol Connector_Generic:Conn_01x07 -> Connector_Generic:Conn_02x06_Odd_Even
- Lk4: renamed from J10; footprint Connector_PinHeader_2.54mm:PinHeader_1x02_P2.54mm_Vertical -> Jumper:SolderJumper-2_P1.3mm_Open_RoundedPad1.0x1.5mm
- P12, P13, P14, P15, P17, P6, P9: footprint IoEngineering:CONN_PWR_2P_3.5MM -> IoEngineering:CONN_PWR_2P_3.5MM_CAMBLOCK
- P3: footprint Connector_PinHeader_2.54mm:PinHeader_1x06_P2.54mm_Vertical -> Connector_PinHeader_2.54mm:PinHeader_2x05_P2.54mm_Vertical; symbol Connector_Generic:Conn_01x06 -> Connector_Generic:Conn_02x05_Odd_Even
- P8: footprint Connector_PinHeader_2.54mm:PinHeader_1x04_P2.54mm_Vertical -> Connector_PinHeader_2.54mm:PinHeader_2x03_P2.54mm_Vertical; symbol Connector_Generic:Conn_01x04 -> Connector_Generic:Conn_02x03_Odd_Even
- renumbered J4 to Lk1, J8 to Lk2, J7 to Lk3
Connections:
- net 3V3: now also P11.2 (Pin_2)
- net CS: now also P3.1 (Pin_1); no longer P3.2 (Pin_2)
- net GND: now also P3.10 (Pin_10), P3.2 (Pin_2), P3.4 (Pin_4), P3.6 (Pin_6), P3.8 (Pin_8), P8.2 (Pin_2), P8.4 (Pin_4), P8.6 (Pin_6), P11.1 (Pin_1), P11.3 (Pin_3); no longer P3.1 (Pin_1), P8.1 (Pin_1)
- net LimX: now also P8.5 (Pin_5); no longer P8.4 (Pin_4)
- net LimZ: now also P8.1 (Pin_1); no longer P8.2 (Pin_2)
- net PB2: now also J9.1 (Pin_1); no longer J9.2 (Pin_2)
- net PB3: now also J14.2 (Pin_2), J16.2 (Pin_2); no longer J14.1, J16.1
- net PB5: now also J16.1 (Pin_1); no longer J16.2
- net PC4: now also J15.2 (Pin_2); no longer J15.1
- net PC7: now also J12.1 (Pin_1), J14.1 (Pin_1); no longer J12.2, J14.2
- net PD0: now also J15.1 (Pin_1); no longer J15.2
- net PE0: now also J12.2 (Pin_2), J13.2 (Pin_2); no longer J12.1, J13.1
- net PF1: now also J13.1 (Pin_1); no longer J13.2
- net Probe: now also P3.9 (Pin_9); no longer P3.6 (Pin_6)
- net Reset: now also P3.7 (Pin_7); no longer P3.5 (Pin_5)
- net SD: now also P3.5 (Pin_5); no longer P3.4 (Pin_4)
- net VBUS: now also P11.4 (Pin_4)
- net at A1.5 (B1), P6.1 (Pin_1): now also P4.4 (Pin_4)
- net at A1.6 (B2), P6.2 (Pin_2): now also P4.3 (Pin_3)
- net at Lk3.2 (Pin_2), Q1.2 (S), Q2.2 (S)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: now also J9.10 (Pin_10), J9.12 (Pin_12), J9.2 (Pin_2), J9.4 (Pin_4), J9.6 (Pin_6), J9.8 (Pin_8); no longer J9.1 (Pin_1)
- net at Q1.3 (D): now also J9.9 (Pin_9); no longer J9.6 (Pin_6)
- net at A1.4 (A1), P9.1 (Pin_1): now also P4.2 (Pin_2)
- net at A1.3 (A2), P9.2 (Pin_2): now also P4.1 (Pin_1)
- net at A2.3 (A2), P12.2 (Pin_2): now also P5.1 (Pin_1)
- net at A2.4 (A1), P12.1 (Pin_1): now also P5.2 (Pin_2)
- net at A2.5 (B1), P13.1 (Pin_1): now also P5.4 (Pin_4)
- net at A2.6 (B2), P13.2 (Pin_2): now also P5.3 (Pin_3)
- net at A3.3 (A2), P14.2 (Pin_2): now also P10.1 (Pin_1)
- net at A3.4 (A1), P14.1 (Pin_1): now also P10.2 (Pin_2)
- net at A3.5 (B1), P15.1 (Pin_1): now also P10.4 (Pin_4)
- net at A3.6 (B2), P15.2 (Pin_2): now also P10.3 (Pin_3)
- net at Q4.3 (D): now also J9.7 (Pin_7); no longer J9.5 (Pin_5)
- net at Q3.3 (D): now also J9.5 (Pin_5); no longer J9.4 (Pin_4)
- net at Lk2.1 (Pin_1): now also J9.11 (Pin_11); no longer J9.7 (Pin_7)
Other:
- moved on the sheet: A1, A2, A3, C4, C5, J1, J11, J2, J3, J5, J6, Lk1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
