File: design Trinamic TMC2130 version/CNC Boosterpack.sch (KiCad schematic (older format))
At the start: 69 parts, among them J1 SBW, J10 EEPROMaddr, J11 UART/GPIO, J4 I2CDrv, J5 I2C, J6 RESET, J7 VDrvGND, J8 VDrvSel, J9 Spindle/Coolant, P1 CONN_02x10, P10 XC, P12 YA, P13 YB, P14 ZA, P15 ZB, P17 VMOT, P2 GPIO, P3 Control, P4 ZC, P5 YC, P6 XB, P7 CONN_02x10, P8 Limits, P9 XA, Q1 2N7002, Q2 2N7002, Q3 2N7002, Q4 2N7002, U1 TLP290-4, U2 TLP290-4, U3 TLP290-4, U4 24LC16, U5 TCA9406, U6 MSP430G2553-20

Commit message: Updated to latest revision
A small batch of the Trinamic-version PCB has been made, driver
development in good progress. Marlin-style M-commands will be supported
including status reports. Grbl protocol extensions allows real-trime
plotting of data (stallguard value) for simpler tuning.
Parts:
- removed A1, A2, A3: Pololu_Breakout_DRV8825, IoEngineering:Polulu_A4988, symbol Driver_Motor:Pololu_Breakout_DRV8825
- removed P10: XC, Connector_PinSocket_2.54mm:PinSocket_1x02_P2.54mm_Vertical, symbol Connector_Generic:Conn_01x02
- removed P4: ZC, Connector_PinSocket_2.54mm:PinSocket_1x02_P2.54mm_Vertical, symbol Connector_Generic:Conn_01x02
- removed P5: YC, Connector_PinSocket_2.54mm:PinSocket_1x02_P2.54mm_Vertical, symbol Connector_Generic:Conn_01x02
- removed R10, R11, R12, R13, R14: 0R, Resistor_SMD:R_0805_2012Metric, symbol Device:R
- added A1, A2, A3: SilentStepStick_Breakout_TMC2130, IoEngineering:SilentStepStick_TMC2130, symbol IoEngineering:SilentStepStick_Breakout_TMC2130
- added J12, J13, J14, J2, J3: Lk, Jumper:SolderJumper-2_P1.3mm_Open_RoundedPad1.0x1.5mm, symbol Connector_Generic:Conn_01x02
- added P10: YMotor, IoEngineering:PinHeader_1x04_P2.54mm_Vertical_Motor, symbol Connector_Generic:Conn_01x04
- added P11: Power, Connector_PinHeader_2.54mm:PinHeader_2x02_P2.54mm_Vertical, symbol Connector_Generic:Conn_02x02_Odd_Even
- added P4: XMotor, IoEngineering:PinHeader_1x04_P2.54mm_Vertical_Motor, symbol Connector_Generic:Conn_01x04
- added P5: ZMotor, IoEngineering:PinHeader_1x04_P2.54mm_Vertical_Motor, symbol Connector_Generic:Conn_01x04
- C6: value 100n -> 1n
- J9: footprint Connector_PinHeader_2.54mm:PinHeader_1x07_P2.54mm_Vertical -> Connector_PinHeader_2.54mm:PinHeader_2x06_P2.54mm_Vertical; symbol Connector_Generic:Conn_01x07 -> Connector_Generic:Conn_02x06_Odd_Even
- Lk4: renamed from J10; footprint Connector_PinHeader_2.54mm:PinHeader_1x02_P2.54mm_Vertical -> Jumper:SolderJumper-2_P1.3mm_Open_RoundedPad1.0x1.5mm
- P1: value CONN_02x10 -> BP A-B
- P12, P13, P14, P15, P17, P6, P9: footprint IoEngineering:CONN_PWR_2P_3.5MM -> IoEngineering:CONN_PWR_2P_3.5MM_CAMBLOCK
- P3: footprint Connector_PinHeader_2.54mm:PinHeader_1x06_P2.54mm_Vertical -> Connector_PinHeader_2.54mm:PinHeader_2x05_P2.54mm_Vertical; symbol Connector_Generic:Conn_01x06 -> Connector_Generic:Conn_02x05_Odd_Even
- P7: value CONN_02x10 -> BP C-D
- P8: footprint Connector_PinHeader_2.54mm:PinHeader_1x04_P2.54mm_Vertical -> Connector_PinHeader_2.54mm:PinHeader_2x03_P2.54mm_Vertical; symbol Connector_Generic:Conn_01x04 -> Connector_Generic:Conn_02x03_Odd_Even
- renumbered J4 to Lk1, J8 to Lk2, J7 to Lk3
Connections:
- net CS: now also P3.1 (Pin_1); no longer P3.2 (Pin_2)
- net ENX: now also A1.11 (~EN)
- net ENY: now also A2.11 (~EN)
- net ENZ: now also A3.11 (~EN)
- net GND: now also P3.10 (Pin_10), P3.2 (Pin_2), P3.4 (Pin_4), P3.6 (Pin_6), P3.8 (Pin_8), P8.2 (Pin_2), P8.4 (Pin_4), P8.6 (Pin_6), A1.1 (GND), A1.7 (GND), A2.1 (GND), A2.7 (GND), A3.1 (GND), A3.7 (GND), P11.1 (Pin_1), P11.3 (Pin_3); no longer P3.1 (Pin_1), P8.1 (Pin_1)
- net LimX: now also P8.5 (Pin_5); no longer P8.4 (Pin_4)
- net LimZ: now also P8.1 (Pin_1); no longer P8.2 (Pin_2)
- net PB2: now also J9.1 (Pin_1); no longer J9.2 (Pin_2)
- net PB3: now also J14.1 (Pin_1), J2.1 (Pin_1)
- net PB4: now also A3.18 (DIR)
- net PB5: now also J2.2 (Pin_2)
- net PB6: now also A2.18 (DIR)
- net PB7: now also A1.18 (DIR)
- net PC4: now also J3.1 (Pin_1)
- net PC7: now also J12.2 (Pin_2), J14.2 (Pin_2)
- net PD0: now also J3.2 (Pin_2)
- net PD1: now also A1.17 (STEP)
- net PD2: now also A2.17 (STEP)
- net PD3: now also A3.17 (STEP)
- net PE0: now also J12.1 (Pin_1), J13.1 (Pin_1)
- net PF0: now also U6.8 (P2.0)
- net PF1: now also J13.2 (Pin_2)
- net Probe: now also P3.9 (Pin_9); no longer P3.6 (Pin_6)
- net Reset: now also P3.7 (Pin_7); no longer P3.5 (Pin_5)
- net SCK: now also A1.13 (SCK), A2.13 (SCK), A3.13 (SCK)
- net SD: now also P3.5 (Pin_5); no longer P3.4 (Pin_4)
- net SDI: now also U6.4 (P1.2), A1.12 (SDI), A2.12 (SDI), A3.12 (SDI); no longer U6.3 (P1.1)
- net SDO: now also U6.3 (P1.1), A1.15 (SDO), A2.15 (SDO), A3.15 (SDO); no longer U6.4 (P1.2)
- net VBUS: now also P11.4 (Pin_4)
- net ~CSX: now also A1.14 (CS)
- net ~CSY: now also A2.14 (CS)
- net ~CSZ: now also A3.14 (CS)
- net at P6.1 (Pin_1): now also A1.5 (B1), P4.4 (Pin_4)
- net at P6.2 (Pin_2): now also A1.6 (B2), P4.3 (Pin_3)
- net at Lk3.2 (Pin_2), Q1.2 (S), Q2.2 (S)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: now also J9.10 (Pin_10), J9.12 (Pin_12), J9.2 (Pin_2), J9.4 (Pin_4), J9.6 (Pin_6), J9.8 (Pin_8); no longer J9.1 (Pin_1)
- net at Q1.3 (D): now also J9.9 (Pin_9); no longer J9.6 (Pin_6)
- net at P9.1 (Pin_1): now also A1.4 (A1), P4.2 (Pin_2)
- net at P9.2 (Pin_2): now also A1.3 (A2), P4.1 (Pin_1)
- net at P12.2 (Pin_2): now also A2.3 (A2), P10.1 (Pin_1)
- net at P12.1 (Pin_1): now also A2.4 (A1), P10.2 (Pin_2)
- net at P13.1 (Pin_1): now also A2.5 (B1), P10.4 (Pin_4)
- net at P13.2 (Pin_2): now also A2.6 (B2), P10.3 (Pin_3)
- net at P14.2 (Pin_2): now also A3.3 (A2), P5.1 (Pin_1)
- net at P14.1 (Pin_1): now also A3.4 (A1), P5.2 (Pin_2)
- net at P15.1 (Pin_1): now also A3.5 (B1), P5.4 (Pin_4)
- net at P15.2 (Pin_2): now also A3.6 (B2), P5.3 (Pin_3)
- net at Q4.3 (D): now also J9.7 (Pin_7); no longer J9.5 (Pin_5)
- net at Q3.3 (D): now also J9.5 (Pin_5); no longer J9.4 (Pin_4)
- net at Lk2.1 (Pin_1): now also J9.11 (Pin_11); no longer J9.7 (Pin_7)
- net DIAGY: now reaches U6.5 (P1.3)
- net DIAGY: now also A2.9 (DIAG1)
- net DIAGX: now reaches U6.7 (P1.5)
- net DIAGX: now also A1.9 (DIAG1)
- net 3V3 renamed +3V3
- net +3V3: now also A1.2 (VIO), A2.2 (VIO), A3.2 (VIO), P11.2 (Pin_2)
- net DIAG renamed DIAGZ
- net DIAGZ: now also A3.9 (DIAG1)
- net VCCB renamed VCCQ
- net VMOT renamed VDDF
- net VDDF: now also A1.8 (VMOT), A2.8 (VMOT), A3.8 (VMOT)
Other:
- moved on the sheet: Lk3, P12, P13, P14, P15, P6, P9
