File: motor driver/Motor driver dummy.kicad_pcb (KiCad board)
At the start: 2 copper layers, 15 x 20.5 mm, 9 parts, among them P1 CONN_01X08, P2 CONN_01X08, Q1 2N7002, Q2 2N7002, Q3 2N7002

Commit message: Updated motor driver dummy to KiCad v5 format
Parts:
- P1, P2: footprint Pin_Headers:Pin_Header_Straight_1x08_Pitch2.54mm -> Connector_PinHeader_2.54mm:PinHeader_1x08_P2.54mm_Vertical
- Q1, Q2, Q3: footprint TO_SOT_Packages_SMD:SOT-23 -> Package_TO_SOT_SMD:SOT-23
- R1, R2, R3, R4: footprint Resistors_SMD:R_0805 -> Resistor_SMD:R_0805_2012Metric
