File: motor driver/Motor driver dummy.sch (KiCad schematic (older format))
At the start: 9 parts, among them P1 CONN_01X08, P2 CONN_01X08, Q1 2N7002, Q2 2N7002, Q3 2N7002

Commit message: Updated motor driver dummy to KiCad v5 format
Parts:
- P1, P2: footprint Pin_Headers:Pin_Header_Straight_1x08_Pitch2.54mm -> Connector_PinHeader_2.54mm:PinHeader_1x08_P2.54mm_Vertical; symbol CONN_01X08 -> Connector_Generic:Conn_01x08
- Q1, Q2, Q3: footprint TO_SOT_Packages_SMD:SOT-23 -> Package_TO_SOT_SMD:SOT-23; symbol MMBF170 -> Transistor_FET:2N7002
- R1, R2, R3, R4: footprint Resistors_SMD:R_0805 -> Resistor_SMD:R_0805_2012Metric; symbol R -> device:R
Connections:
- wire segments 17 -> 26
- no-connect marks 0 -> 7
Other:
- moved on the sheet: Q1, Q2, Q3
Changed lines of the file:
@@
-EESchema Schematic File Version 2
-LIBS:power
-LIBS:device
-LIBS:switches
-LIBS:relays
-LIBS:transistors
-LIBS:conn
-LIBS:linear
-LIBS:regul
-LIBS:engineering
+EESchema Schematic File Version 4
 LIBS:Motor driver dummy-cache
-EELAYER 25 0
+EELAYER 29 0
 EELAYER END
 $Descr A4 11693 8268
@@
 Sheet 1 1
 Title "Polulu style driver i/f for external drivers like DQ542MA "
-Date "2018-04-17"
+Date "2021-10-28"
 Rev "1"
 Comp "Io Engineering"
@@
 $EndDescr
 $Comp
-L MMBF170 Q3
+L Transistor_FET:2N7002 Q3
 U 1 1 5AD33A56
-P 6750 3800
-F 0 "Q3" H 6950 3875 50  0000 L CNN
-F 1 "2N7002" H 6950 3800 50  0000 L CNN
-F 2 "TO_SOT_Packages_SMD:SOT-23" H 6950 3725 50  0001 L CIN
-F 3 "" H 6750 3800 50  0000 L CNN
-	1    6750 3800
-	1    0    0    -1
-$EndComp
-$Comp
-L MMBF170 Q2
+P 6750 3850
+F 0 "Q3" H 6950 3925 50  0000 L CNN
+F 1 "2N7002" H 6950 3850 50  0000 L CNN
+F 2 "Package_TO_SOT_SMD:SOT-23" H 6950 3775 50  0001 L CIN
+F 3 "" H 6750 3850 50  0000 L CNN
+	1    6750 3850
+	1    0    0    -1
+$EndComp
+$Comp
+L Transistor_FET:2N7002 Q2
 U 1 1 5AD33B0B
-P 5600 3800
-F 0 "Q2" H 5800 3875 50  0000 L CNN
-F 1 "2N7002" H 5800 3800 50  0000 L CNN
-F 2 "TO_SOT_Packages_SMD:SOT-23" H 5800 3725 50  0001 L CIN
-F 3 "" H 5600 3800 50  0000 L CNN
-	1    5600 3800
-	1    0    0    -1
-$EndComp
-$Comp
-L MMBF170 Q1
+P 5600 3850
+F 0 "Q2" H 5800 3925 50  0000 L CNN
+F 1 "2N7002" H 5800 3850 50  0000 L CNN
+F 2 "Package_TO_SOT_SMD:SOT-23" H 5800 3775 50  0001 L CIN
+F 3 "" H 5600 3850 50  0000 L CNN
+	1    5600 3850
+	1    0    0    -1
+$EndComp
+$Comp
+L Transistor_FET:2N7002 Q1
 U 1 1 5AD33B44
-P 4400 3800
-F 0 "Q1" H 4600 3875 50  0000 L CNN
-F 1 "2N7002" H 4600 3800 50  0000 L CNN
-F 2 "TO_SOT_Packages_SMD:SOT-23" H 4600 3725 50  0001 L CIN
-F 3 "" H 4400 3800 50  0000 L CNN
-	1    4400 3800
-	1    0    0    -1
-$EndComp
-$Comp
-L R R3
+P 4400 3850
+F 0 "Q1" H 4600 3925 50  0000 L CNN
+F 1 "2N7002" H 4600 3850 50  0000 L CNN
+F 2 "Package_TO_SOT_SMD:SOT-23" H 4600 3775 50  0001 L CIN
+F 3 "" H 4400 3850 50  0000 L CNN
+	1    4400 3850
+	1    0    0    -1
+$EndComp
+$Comp
+L device:R R3
 U 1 1 5AD33B90
 P 6450 4100
 F 0 "R3" V 6530 4100 50  0000 C CNN
 F 1 "10K" V 6450 4100 50  0000 C CNN
-F 2 "Resistors_SMD:R_0805" V 6380 4100 50  0001 C CNN
+F 2 "Resistor_SMD:R_0805_2012Metric" V 6380 4100 50  0001 C CNN
 F 3 "" H 6450 4100 50  0001 C CNN
 	1    6450 4100
@@
 $EndComp
 $Comp
-L R R2
+L device:R R2
 U 1 1 5AD33C03
 P 5300 4100
 F 0 "R2" V 5380 4100 50  0000 C CNN
 F 1 "10K" V 5300 4100 50  0000 C CNN
-F 2 "Resistors_SMD:R_0805" V 5230 4100 50  0001 C CNN
+F 2 "Resistor_SMD:R_0805_2012Metric" V 5230 4100 50  0001 C CNN
 F 3 "" H 5300 4100 50  0001 C CNN
 	1    5300 4100
@@
 $EndComp
 $Comp
-L R R1
+L device:R R1
 U 1 1 5AD33C22
 P 4100 4100
 F 0 "R1" V 4180 4100 50  0000 C CNN
 F 1 "10K" V 4100 4100 50  0000 C CNN
-F 2 "Resistors_SMD:R_0805" V 4030 4100 50  0001 C CNN
+F 2 "Resistor_SMD:R_0805_2012Metric" V 4030 4100 50  0001 C CNN
 F 3 "" H 4100 4100 50  0001 C CNN
 	1    4100 4100
@@
 $EndComp
 $Comp
-L CONN_01X08 P2
+L Connector_Generic:Conn_01x08 P2
 U 1 1 5AD33C83
-P 3600 3900
-F 0 "P2" H 3600 4350 50  0000 C CNN
-F 1 "CONN_01X08" V 3700 3900 50  0000 C CNN
-F 2 "Pin_Headers:Pin_Header_Straight_1x08_Pitch2.54mm" H 3600 3900 50  0001 C CNN
-F 3 "" H 3600 3900 50  0000 C CNN
-	1    3600 3900
+P 3600 3950
+F 0 "P2" H 3600 4400 50  0000 C CNN
+F 1 "CONN_01X08" V 3700 3950 50  0000 C CNN
+F 2 "Connector_PinHeader_2.54mm:PinHeader_1x08_P2.54mm_Vertical" H 3600 3950 50  0001 C CNN
+F 3 "" H 3600 3950 50  0000 C CNN
+	1    3600 3950
 	1    0    0    1
 $EndComp
 $Comp
-L CONN_01X08 P1
+L Connector_Generic:Conn_01x08 P1
 U 1 1 5AD33CE9
-P 2600 3900
-F 0 "P1" H 2600 4350 50  0000 C CNN
-F 1 "CONN_01X08" V 2700 3900 50  0000 C CNN
-F 2 "Pin_Headers:Pin_Header_Straight_1x08_Pitch2.54mm" H 2600 3900 50  0001 C CNN
-F 3 "" H 2600 3900 50  0000 C CNN
-	1    2600 3900
+P 2600 3950
+F 0 "P1" H 2600 4400 50  0000 C CNN
+F 1 "CONN_01X08" V 2700 3950 50  0000 C CNN
+F 2 "Connector_PinHeader_2.54mm:PinHeader_1x08_P2.54mm_Vertical" H 2600 3950 50  0001 C CNN
+F 3 "" H 2600 3950 50  0000 C CNN
+	1    2600 3950
 	-1   0    0    1
 $EndComp
@@
 	3400 3550 3100 3550
 Wire Wire Line
-	3100 3550 3100 4500
-Wire Wire Line
-	3100 4400 6850 4400
-Wire Wire Line
-	6850 4400 6850 4000
+	3100 3550 3100 4400
+Wire Wire Line
+	3100 4400 4100 4400
 Text Label 4000 3850 2    60   ~ 0
 ~EN
@@
 STEP
 Wire Wire Line
-	6550 3850 6350 3850
+	6550 3850 6450 3850
 Wire Wire Line
 	6450 3850 6450 3950
@@
 Connection ~ 6450 4400
 Wire Wire Line
-	5400 3850 5200 3850
+	5400 3850 5300 3850
 Wire Wire Line
 	5300 3850 5300 3950
@@
 Connection ~ 5300 4400
 Wire Wire Line
-	4000 3850 4200 3850
+	4000 3850 4100 3850
 Wire Wire Line
 	4100 3850 4100 3950
@@
 	4100 4250 4100 4400
 Connection ~ 4100 4400
-Wire Wire Line
-	5700 4000 5700 4400
-Connection ~ 5700 4400
-Wire Wire Line
-	4500 4000 4500 4400
-Connection ~ 4500 4400
-Text Label 4500 3600 0    60   ~ 0
+Text Label 4500 3650 0    60   ~ 0
 EN
-Text Label 5700 3600 0    60   ~ 0
+Text Label 5700 3650 0    60   ~ 0
 ~STEP
-Text Label 6850 3600 0    60   ~ 0
+Text Label 6850 3650 0    60   ~ 0
 ~DIR
 $Comp
-L GND #PWR01
+L power1:GND #PWR01
 U 1 1 5AD35459
 P 3100 4500
@@
 Connection ~ 3100 4400
 $Comp
-L R R4
+L device:R R4
 U 1 1 5AD35617
 P 3200 4100
 F 0 "R4" V 3280 4100 50  0000 C CNN
 F 1 "0R" V 3200 4100 50  0000 C CNN
-F 2 "Resistors_SMD:R_0805" V 3130 4100 50  0001 C CNN
+F 2 "Resistor_SMD:R_0805_2012Metric" V 3130 4100 50  0001 C CNN
 F 3 "" H 3200 4100 50  0001 C CNN
 	1    3200 4100
@@
 Wire Wire Line
 	3200 3950 3400 3950
+Wire Wire Line
+	6450 3850 6350 3850
+Wire Wire Line
+	6450 4400 6850 4400
+Wire Wire Line
+	5300 3850 5200 3850
+Wire Wire Line
+	4100 3850 4200 3850
+Wire Wire Line
+	3100 4400 3100 4500
+NoConn ~ 2800 3750
+NoConn ~ 2800 3850
+NoConn ~ 2800 3950
+NoConn ~ 2800 4050
+NoConn ~ 2800 4150
+NoConn ~ 3400 3650
+NoConn ~ 3400 4150
+Wire Wire Line
+	5300 4400 5700 4400
+Wire Wire Line
+	4100 4400 4500 4400
+Wire Wire Line
+	6850 4050 6850 4400
+Wire Wire Line
+	5700 4050 5700 4400
+Connection ~ 5700 4400
+Wire Wire Line
+	5700 4400 6450 4400
+Wire Wire Line
+	4500 4050 4500 4400
+Connection ~ 4500 4400
+Wire Wire Line
+	4500 4400 5300 4400
 $EndSCHEMATC
